Commit message: Finished garry urdf file

File: urdf/garry.urdf.xacro (robot description, xacro)
@@ -1,86 +1,159 @@
-<?xml version="1.0" encoding="utf-8"?>
-<!-- =================================================================================== -->
-<!-- |    This document was autogenerated by xacro from garry.urdf                     | -->
-<!-- |    EDITING THIS FILE BY HAND IS NOT RECOMMENDED                                 | -->
-<!-- =================================================================================== -->
-<robot name="garry" xmlns:xacro="http://www.ros.org/wiki/xacro">
-  <!-- materials  -->
-  <material name="black">
-    <color rgba="0 0 0 0"/>
-  </material>
-  <material name="blue">
-    <color rgba="0 0 0.8 1"/>
-  </material>
-  <!-- links -->
-  <link name="base_link">
-    <visual>
-      <geometry>
-        <box size="24.5 17.0 1.25"/>
-      </geometry>
-      <origin xyz="0 0 0"/>
-    </visual>
-    <collision>
-      <geometry>
-        <box size="24.5 17.0 1.25"/>
-      </geometry>
-    </collision>
-  </link>
-  <link name="boards_link">
-    <visual>
-      <geometry>
-        <box size="7.0 8.0 15.0"/>
-      </geometry>
-      <origin xyz="0.0 0.0 7.5625"/>
-    </visual>
-    <collision>
-      <geometry>
-        <box size="7.0 8.0 1.5"/>
-      </geometry>
-    </collision>
-  </link>
-  <joint name="base_to_board" type="fixed">
-    <parent link="base_link"/>
-    <child link="boards_link"/>
-    <origin xyz="-2.25 0.0 0.6125"/>
-  </joint>
-  <link name="right_wheel">
-    <visual>
-      <origin xyz="-3.25 5.5 -2.3125"/>
-      <origin rpy="1.0 1.0 1.0"/>
-      <geometry>
-        <cylinder length="1.0" radius="2.7"/>
-      </geometry>
-    </visual>
-    <collision>
-      <geometry>
-        <cylinder length="1.0" radius="2.7"/>
-      </geometry>
-    </collision>
-  </link>
-  <joint name="base_to_right_wheel" type="fixed">
-    <parent link="base_link"/>
-    <child link="right_wheel"/>
-    <origin xyz="-3.25.0 5.5 -0.6125"/>
-  </joint>
-  <!-->
-	<link name="left_wheel">
+<?xml version="1.0"?>
+<robot xmlns:xacro="http://www.ros.org/wiki/xacro" name="garry">
+	<xacro:property name="base_x_len" value="17.0"/>
+	<xacro:property name="base_y_len" value="25.0"/>
+	<xacro:property name="base_z_len" value="0.4"/>
+	<xacro:property name="board_y_back" value="3.5"/>
+	<xacro:property name="board_x_len" value="7.0"/>
+	<xacro:property name="board_y_len" value="9.0"/>
+	<xacro:property name="board_z_len" value="15.0"/>
+	<xacro:property name="board_y_origin" value="${-(base_y_len/2-board_y_back-board_y_len/2)}"/>
+	<xacro:property name="wheel_d" value="5.4"/>
+	<xacro:property name="wheel_th" value="1.8"/>
+	<xacro:property name="wheel_y_origin" value="${board_y_origin}"/>
+	<xacro:property name="wheel_x_origin" value="5.5"/>
+	<xacro:property name="wheel_z_origin" value="${-wheel_d/2-1.5*base_z_len}"/>
+	<xacro:property name="gearbox_x_origin" value="2.6"/>
+	<xacro:property name="gearbox_x_len" value="2.15"/>
+	<xacro:property name="gearbox_z_len" value="4.2"/>
+	<xacro:property name="gearbox_x_joint" value="${gearbox_x_origin+gearbox_x_len/2+wheel_th/2}"/>
+	<xacro:property name="gearbox_z_origin" value="${-gearbox_z_len/2-base_z_len}"/>
+	<xacro:property name="imu_x_origin" value="-4.0"/>
+	<xacro:property name="imu_x_len" value="1.7"/>
+	<xacro:property name="imu_y_len" value="2.2"/>
+	<xacro:property name="imu_z_len" value="0.1"/>
+	<xacro:property name="raspi_cam_z_origin" value="15.0"/>
+	<xacro:property name="webcam_x_origin" value="1.6"/>
+	<xacro:property name="webcam_y_origin" value="${-(base_y_len/2-board_y_back)}"/>
+	<xacro:property name="webcam_z_origin" value="${raspi_cam_z_origin}"/>
+	<link name="base_link">
 		<visual>
-			<origin rpy="220.0 -85.0 -2.5125"/>
 			<geometry>
-				<cylinder length="1.0" radius="-2.5125"/>
+				<box size="${base_x_len} ${base_y_len} ${base_z_len}"/>
 			</geometry>
-			<material name="black"/>
 		</visual>
 		<collision>
 			<geometry>
-				<cylinder length="1.0" radius="2.5125"/>
+				<box size="${base_x_len} ${base_y_len} ${base_z_len}"/>
 			</geometry>
 		</collision>
 	</link>
-	<joint name="base_to_left_wheel" type="fixed">
+	<link name="boards_link">
+		<visual>
+			<geometry>
+				<box size="${board_x_len} ${board_y_len} ${board_z_len}"/>
+			</geometry>
+		</visual>
+		<collision>
+			<geometry>
+				<box size="${board_x_len} ${board_y_len} ${board_z_len}"/>
+			</geometry>
+		</collision>
+	</link>
+	<joint name="base_to_board" type="fixed">
 		<parent link="base_link"/>
+		<child link="boards_link"/>
+		<origin xyz="0.0 ${board_y_origin} ${board_z_len/2}"/>
+	</joint>
+	<link name="right_gearbox">
+		<visual>
+			<origin xyz="${gearbox_x_origin} ${wheel_y_origin} ${gearbox_z_origin}"/>
+			<geometry>
+				<box size="${gearbox_x_len} ${wheel_d} ${gearbox_z_len}"/>
+			</geometry>
+		</visual>
+		<collision>
+			<geometry>
+				<box size="${gearbox_x_len} ${wheel_d} ${gearbox_z_len}"/>
+			</geometry>
+		</collision>
+	</link>
+	<link name="left_gearbox">
+		<visual>
+			<origin xyz="${-gearbox_x_origin} ${wheel_y_origin} ${gearbox_z_origin}"/>
+			<geometry>
+				<box size="${gearbox_x_len} ${wheel_d} ${gearbox_z_len}"/>
+			</geometry>
+		</visual>
+		<collision>
+			<geometry>
+				<box size="${gearbox_x_len} ${wheel_d} ${gearbox_z_len}"/>
+			</geometry>
+		</collision>
+	</link>
+	<link name="right_wheel">
+		<visual>
+			<origin rpy="${pi/2} 0.0 ${pi/2} "/>
+			<geometry>
+				<cylinder length="${wheel_th}" radius="${wheel_d/2}"/>
+			</geometry>
+		</visual>
+		<collision>
+			<geometry>
+				<cylinder length="${wheel_th}" radius="${wheel_d/2}"/>
+			</geometry>
+		</collision>
+	</link>
+	<link name="left_wheel">
+		<visual>
+			<origin rpy="${pi/2} 0.0 ${pi/2} "/>
+			<geometry>
+				<cylinder length="${wheel_th}" radius="${wheel_d/2}"/>
+			</geometry>
+		</visual>
+		<collision>
+			<geometry>
+				<cylinder length="${wheel_th}" radius="${wheel_d/2}"/>
+			</geometry>
+		</collision>
+	</link>
+	<joint name="left_wheel_to_left_gearbox" type="fixed">
+		<parent link="left_gearbox"/>
 		<child link="left_wheel"/>
-		<origin xyz="220.0 -85.0 -2.5125"/>
+		<origin xyz="${-gearbox_x_joint} ${wheel_y_origin} ${wheel_z_origin}"/>
 	</joint>
-<-->
+	<joint name="left_gearbox_to_base" type="fixed">
+		<parent link="base_link"/>
+		<child link="left_gearbox"/>
+		<origin xyz="${-gearbox_x_origin} ${wheel_y_origin} ${base_z_len/2}"/>
+	</joint>
+	<joint name="right_wheel_to_right_gearbox" type="fixed">
+		<parent link="right_gearbox"/>
+		<child link="right_wheel"/>
+		<origin xyz="${gearbox_x_joint} ${wheel_y_origin} ${wheel_z_origin}"/>
+	</joint>
+	<joint name="right_gearbox_to_base" type="fixed">
+		<parent link="base_link"/>
+		<child link="right_gearbox"/>
+		<origin xyz="${gearbox_x_origin} ${wheel_y_origin} ${base_z_len/2}"/>
+	</joint>
+	<link name="imu_link">
+		<visual>
+			<geometry>
+				<box size="${imu_x_len} ${imu_y_len} ${imu_z_len}"/>
+			</geometry>
+		</visual>
+		<collision>
+			<geometry>
+				<box size="${imu_x_len} ${imu_y_len} ${imu_z_len}"/>
+			</geometry>
+		</collision>
+	</link>
+	<joint name="imu_to_base" type="fixed">
+		<parent link="base_link"/>
+		<child link="imu_link"/>
+		<origin xyz="${imu_x_origin} ${wheel_y_origin} ${base_z_len/2}"/>
+	</joint>
+	<link name="raspi_cam_link"/>
+	<joint name="raspi_cam_to_base" type="fixed">
+		<parent link="base_link"/>
+		<child link="raspi_cam_link"/>
+		<origin xyz="0.0 0.0 ${raspi_cam_z_origin}"/>
+	</joint>
+	<link name="webcam_link"/>
+	<joint name="webcam_to_base" type="fixed">
+		<parent link="base_link"/>
+		<child link="webcam_link"/>
+		<origin xyz="${webcam_x_origin} ${webcam_y_origin} ${webcam_z_origin}"/>
+	</joint>
 </robot>

Commit message: added state publisher

File: urdf/garry.urdf.xacro (robot description, xacro)
@@ -108,8 +108,9 @@
 		</collision>
 	</link>
-	<joint name="left_wheel_to_left_gearbox" type="fixed">
+	<joint name="left_wheel_to_left_gearbox" type="continuous">
 		<parent link="left_gearbox"/>
 		<child link="left_wheel"/>
 		<origin xyz="${-gearbox_x_joint} ${wheel_y_origin} ${wheel_z_origin}"/>
+		<axis xyz="-1 0 0"/>
 	</joint>
 	<joint name="left_gearbox_to_base" type="fixed">
@@ -118,8 +119,9 @@
 		<origin xyz="${-gearbox_x_origin} ${wheel_y_origin} ${base_z_len/2}"/>
 	</joint>
-	<joint name="right_wheel_to_right_gearbox" type="fixed">
+	<joint name="right_wheel_to_right_gearbox" type="continuous">
 		<parent link="right_gearbox"/>
 		<child link="right_wheel"/>
 		<origin xyz="${gearbox_x_joint} ${wheel_y_origin} ${wheel_z_origin}"/>
+		<axis xyz="-1 0 0"/>
 	</joint>
 	<joint name="right_gearbox_to_base" type="fixed">

Commit message: Fixed wheels und and imu position

File: urdf/garry.urdf.xacro (robot description, xacro)
@@ -23,4 +23,5 @@
 	<xacro:property name="imu_y_len" value="2.2"/>
 	<xacro:property name="imu_z_len" value="0.1"/>
+	<xacro:property name="imu_yaw" value="${-pi/2}"/>
 	<xacro:property name="raspi_cam_z_origin" value="15.0"/>
 	<xacro:property name="webcam_x_origin" value="1.6"/>
@@ -108,5 +109,5 @@
 		</collision>
 	</link>
-	<joint name="left_wheel_to_left_gearbox" type="continuous">
+	<joint name="left_wheel_to_left_gearbox" type="fixed">
 		<parent link="left_gearbox"/>
 		<child link="left_wheel"/>
@@ -119,5 +120,5 @@
 		<origin xyz="${-gearbox_x_origin} ${wheel_y_origin} ${base_z_len/2}"/>
 	</joint>
-	<joint name="right_wheel_to_right_gearbox" type="continuous">
+	<joint name="right_wheel_to_right_gearbox" type="fixed">
 		<parent link="right_gearbox"/>
 		<child link="right_wheel"/>
@@ -145,11 +146,5 @@
 		<parent link="base_link"/>
 		<child link="imu_link"/>
-		<origin xyz="${imu_x_origin} ${wheel_y_origin} ${base_z_len/2}" rpy="0.0 0.0 -pi/2"/>
-	</joint>
-	<link name="raspi_cam_link"/>
-	<joint name="raspi_cam_to_base" type="fixed">
-		<parent link="base_link"/>
-		<child link="raspi_cam_link"/>
-		<origin xyz="0.0 0.0 ${raspi_cam_z_origin}"/>
+		<origin xyz="${imu_x_origin} ${wheel_y_origin} ${base_z_len/2}" rpy="0.0 0.0 ${imu_yaw}"/>
 	</joint>
 	<link name="webcam_link"/>
@@ -157,4 +152,10 @@
 		<parent link="base_link"/>
 		<child link="webcam_link"/>
+		<origin xyz="0.0 0.0 ${raspi_cam_z_origin}"/>
+	</joint>
+	<link name="raspicam_link"/>
+	<joint name="raspicam_to_base" type="fixed">
+		<parent link="base_link"/>
+		<child link="raspicam_link"/>
 		<origin xyz="${webcam_x_origin} ${webcam_y_origin} ${webcam_z_origin}"/>
 	</joint>

Commit message: Converted to meters and fixed x-y

File: urdf/garry.urdf.xacro (robot description, xacro)
@@ -1,30 +1,30 @@
 <?xml version="1.0"?>
 <robot xmlns:xacro="http://www.ros.org/wiki/xacro" name="garry">
-	<xacro:property name="base_x_len" value="17.0"/>
-	<xacro:property name="base_y_len" value="25.0"/>
-	<xacro:property name="base_z_len" value="0.4"/>
-	<xacro:property name="board_y_back" value="3.5"/>
-	<xacro:property name="board_x_len" value="7.0"/>
-	<xacro:property name="board_y_len" value="9.0"/>
-	<xacro:property name="board_z_len" value="15.0"/>
-	<xacro:property name="board_y_origin" value="${-(base_y_len/2-board_y_back-board_y_len/2)}"/>
-	<xacro:property name="wheel_d" value="5.4"/>
-	<xacro:property name="wheel_th" value="1.8"/>
-	<xacro:property name="wheel_y_origin" value="${board_y_origin}"/>
-	<xacro:property name="wheel_x_origin" value="5.5"/>
+	<xacro:property name="base_x_len" value="0.25"/>
+	<xacro:property name="base_y_len" value="0.17"/>
+	<xacro:property name="base_z_len" value="0.004"/>
+	<xacro:property name="board_x_back" value="0.035"/>
+	<xacro:property name="board_y_len" value="0.07"/>
+	<xacro:property name="board_x_len" value="0.09"/>
+	<xacro:property name="board_z_len" value="0.15"/>
+	<xacro:property name="board_x_origin" value="${-(base_x_len/2-board_x_back-board_x_len/2)}"/>
+	<xacro:property name="wheel_d" value="0.054"/>
+	<xacro:property name="wheel_th" value="0.018"/>
+	<xacro:property name="wheel_x_origin" value="${board_x_origin}"/>
+	<xacro:property name="wheel_y_origin" value="0.055"/>
 	<xacro:property name="wheel_z_origin" value="${-wheel_d/2-1.5*base_z_len}"/>
-	<xacro:property name="gearbox_x_origin" value="2.6"/>
-	<xacro:property name="gearbox_x_len" value="2.15"/>
-	<xacro:property name="gearbox_z_len" value="4.2"/>
-	<xacro:property name="gearbox_x_joint" value="${gearbox_x_origin+gearbox_x_len/2+wheel_th/2}"/>
+	<xacro:property name="gearbox_y_origin" value="0.026"/>
+	<xacro:property name="gearbox_y_len" value="0.0215"/>
+	<xacro:property name="gearbox_z_len" value="0.042"/>
+	<xacro:property name="gearbox_y_joint" value="${gearbox_y_origin+gearbox_y_len/2+wheel_th/2}"/>
 	<xacro:property name="gearbox_z_origin" value="${-gearbox_z_len/2-base_z_len}"/>
-	<xacro:property name="imu_x_origin" value="-4.0"/>
-	<xacro:property name="imu_x_len" value="1.7"/>
-	<xacro:property name="imu_y_len" value="2.2"/>
-	<xacro:property name="imu_z_len" value="0.1"/>
-	<xacro:property name="imu_yaw" value="${-pi/2}"/>
-	<xacro:property name="raspi_cam_z_origin" value="15.0"/>
-	<xacro:property name="webcam_x_origin" value="1.6"/>
-	<xacro:property name="webcam_y_origin" value="${-(base_y_len/2-board_y_back)}"/>
+	<xacro:property name="imu_y_origin" value="0.04"/>
+	<xacro:property name="imu_y_len" value="0.017"/>
+	<xacro:property name="imu_x_len" value="0.022"/>
+	<xacro:property name="imu_z_len" value="0.001"/>
+	<xacro:property name="imu_yaw" value="${-pi}"/>
+	<xacro:property name="raspi_cam_z_origin" value="0.15"/>
+	<xacro:property name="webcam_y_origin" value="0.016"/>
+	<xacro:property name="webcam_x_origin" value="${-(base_x_len/2-board_x_back)}"/>
 	<xacro:property name="webcam_z_origin" value="${raspi_cam_z_origin}"/>
 	<link name="base_link">
@@ -55,16 +55,16 @@
 		<parent link="base_link"/>
 		<child link="boards_link"/>
-		<origin xyz="0.0 ${board_y_origin} ${board_z_len/2}"/>
+		<origin xyz="${board_x_origin} 0.0 ${board_z_len/2}"/>
 	</joint>
 	<link name="right_gearbox">
 		<visual>
-			<origin xyz="${gearbox_x_origin} ${wheel_y_origin} ${gearbox_z_origin}"/>
+			<origin xyz="${wheel_x_origin} ${gearbox_y_origin} ${gearbox_z_origin}"/>
 			<geometry>
-				<box size="${gearbox_x_len} ${wheel_d} ${gearbox_z_len}"/>
+				<box size="${wheel_d} ${gearbox_y_len}  ${gearbox_z_len}"/>
 			</geometry>
 		</visual>
 		<collision>
 			<geometry>
-				<box size="${gearbox_x_len} ${wheel_d} ${gearbox_z_len}"/>
+				<box size=" ${wheel_d} ${gearbox_y_len} ${gearbox_z_len}"/>
 			</geometry>
 		</collision>
@@ -72,12 +72,12 @@
 	<link name="left_gearbox">
 		<visual>
-			<origin xyz="${-gearbox_x_origin} ${wheel_y_origin} ${gearbox_z_origin}"/>
+			<origin xyz="${wheel_x_origin} ${-gearbox_y_origin}  ${gearbox_z_origin}"/>
 			<geometry>
-				<box size="${gearbox_x_len} ${wheel_d} ${gearbox_z_len}"/>
+				<box size="${wheel_d} ${gearbox_y_len}  ${gearbox_z_len}"/>
 			</geometry>
 		</visual>
 		<collision>
 			<geometry>
-				<box size="${gearbox_x_len} ${wheel_d} ${gearbox_z_len}"/>
+				<box size="${wheel_d} ${gearbox_y_len}  ${gearbox_z_len}"/>
 			</geometry>
 		</collision>
@@ -85,5 +85,5 @@
 	<link name="right_wheel">
 		<visual>
-			<origin rpy="${pi/2} 0.0 ${pi/2} "/>
+			<origin rpy=" 0.0 ${pi/2} ${pi/2} "/>
 			<geometry>
 				<cylinder length="${wheel_th}" radius="${wheel_d/2}"/>
@@ -98,5 +98,5 @@
 	<link name="left_wheel">
 		<visual>
-			<origin rpy="${pi/2} 0.0 ${pi/2} "/>
+			<origin rpy="0.0 ${pi/2} ${pi/2} "/>
 			<geometry>
 				<cylinder length="${wheel_th}" radius="${wheel_d/2}"/>
@@ -112,5 +112,5 @@
 		<parent link="left_gearbox"/>
 		<child link="left_wheel"/>
-		<origin xyz="${-gearbox_x_joint} ${wheel_y_origin} ${wheel_z_origin}"/>
+		<origin xyz=" ${wheel_x_origin} ${-gearbox_y_joint} ${wheel_z_origin}"/>
 		<axis xyz="-1 0 0"/>
 	</joint>
@@ -118,10 +118,10 @@
 		<parent link="base_link"/>
 		<child link="left_gearbox"/>
-		<origin xyz="${-gearbox_x_origin} ${wheel_y_origin} ${base_z_len/2}"/>
+		<origin xyz=" ${wheel_x_origin} ${-gearbox_y_origin} ${base_z_len/2}"/>
 	</joint>
 	<joint name="right_wheel_to_right_gearbox" type="fixed">
 		<parent link="right_gearbox"/>
 		<child link="right_wheel"/>
-		<origin xyz="${gearbox_x_joint} ${wheel_y_origin} ${wheel_z_origin}"/>
+		<origin xyz="${wheel_x_origin} ${gearbox_y_joint} ${wheel_z_origin}"/>
 		<axis xyz="-1 0 0"/>
 	</joint>
@@ -129,5 +129,5 @@
 		<parent link="base_link"/>
 		<child link="right_gearbox"/>
-		<origin xyz="${gearbox_x_origin} ${wheel_y_origin} ${base_z_len/2}"/>
+		<origin xyz="${wheel_x_origin} ${gearbox_y_origin} ${base_z_len/2}"/>
 	</joint>
 	<link name="imu_link">
@@ -146,5 +146,5 @@
 		<parent link="base_link"/>
 		<child link="imu_link"/>
-		<origin xyz="${imu_x_origin} ${wheel_y_origin} ${base_z_len/2}" rpy="0.0 0.0 ${imu_yaw}"/>
+		<origin xyz=" ${wheel_x_origin} ${imu_y_origin} ${base_z_len/2}" rpy="0.0 0.0 ${imu_yaw}"/>
 	</joint>
 	<link name="webcam_link"/>
@@ -152,5 +152,5 @@
 		<parent link="base_link"/>
 		<child link="webcam_link"/>
-		<origin xyz="0.0 0.0 ${raspi_cam_z_origin}"/>
+		<origin xyz="0.0 ${webcam_y_origin} ${raspi_cam_z_origin}"/>
 	</joint>
 	<link name="raspicam_link"/>
@@ -158,5 +158,5 @@
 		<parent link="base_link"/>
 		<child link="raspicam_link"/>
-		<origin xyz="${webcam_x_origin} ${webcam_y_origin} ${webcam_z_origin}"/>
+		<origin xyz="${webcam_x_origin} 0.0 ${webcam_z_origin}"/>
 	</joint>
 </robot>

Commit message: fixed imu position

File: urdf/garry.urdf.xacro (robot description, xacro)
@@ -19,4 +19,5 @@
 	<xacro:property name="gearbox_y_joint" value="${gearbox_y_origin+gearbox_y_len/2+wheel_th/2}"/>
 	<xacro:property name="gearbox_z_origin" value="${-gearbox_z_len/2-base_z_len}"/>
+    <xacro:property name="imu_x_origin" value="0.00"/>
 	<xacro:property name="imu_y_origin" value="0.04"/>
 	<xacro:property name="imu_y_len" value="0.017"/>
@@ -131,5 +132,5 @@
 		<origin xyz="${wheel_x_origin} ${gearbox_y_origin} ${base_z_len/2}"/>
 	</joint>
-	<link name="imu_link">
+	<link name="base_imu_link">
 		<visual>
 			<geometry>
@@ -145,6 +146,6 @@
 	<joint name="imu_to_base" type="fixed">
 		<parent link="base_link"/>
-		<child link="imu_link"/>
-		<origin xyz=" ${wheel_x_origin} ${imu_y_origin} ${base_z_len/2}" rpy="0.0 0.0 ${imu_yaw}"/>
+		<child link="base_imu_link"/>
+		<origin xyz=" ${imu_x_origin} ${imu_y_origin} ${base_z_len/2}" rpy="0.0 0.0 ${imu_yaw}"/>
 	</joint>
 	<link name="webcam_link"/>

Commit message: fix imu position

File: urdf/garry.urdf.xacro (robot description, xacro)
@@ -24,5 +24,5 @@
 	<xacro:property name="imu_x_len" value="0.022"/>
 	<xacro:property name="imu_z_len" value="0.001"/>
-	<xacro:property name="imu_yaw" value="${-pi}"/>
+	<xacro:property name="imu_yaw" value="${0}"/>
 	<xacro:property name="raspi_cam_z_origin" value="0.15"/>
 	<xacro:property name="webcam_y_origin" value="0.016"/>

Commit message: Fixed IMU position

File: urdf/garry.urdf.xacro (robot description, xacro)
@@ -25,4 +25,5 @@
 	<xacro:property name="imu_z_len" value="0.001"/>
 	<xacro:property name="imu_yaw" value="${0}"/>
+	<xacro:property name="imu_roll" value="${pi}"/>
 	<xacro:property name="raspi_cam_z_origin" value="0.15"/>
 	<xacro:property name="webcam_y_origin" value="0.016"/>
@@ -147,5 +148,5 @@
 		<parent link="base_link"/>
 		<child link="base_imu_link"/>
-		<origin xyz=" ${imu_x_origin} ${imu_y_origin} ${base_z_len/2}" rpy="0.0 0.0 ${imu_yaw}"/>
+		<origin xyz=" ${imu_x_origin} ${imu_y_origin} ${base_z_len/2}" rpy="${imu_roll} 0.0 ${imu_yaw}"/>
 	</joint>
 	<link name="webcam_link"/>
